File: PCB/V2A/ESC-simple_V2A[ervinedit].brd (EAGLE design)
At the start: 40.6 x 95.9 mm, 52 parts, among them IC1 MEGA8-AI, IC2 L6369D, IC3 L6369D, IC4 L6369D, IC6 7805T, Q1 SIRC10DP, Q2 SIRC10DP, Q3 SIRC10DP, Q4 SIRC10DP, Q5 SIRC10DP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

Commit message: replaced paths
Parts:
- moved LED2 1.27 mm to (14.0, 7.94)
Routing:
- net N$15: track 28.8 -> 27.5 mm
- net N$16: track 3.97 -> 5.24 mm
Changed lines of the file:
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@@
 <layer number="21" name="tPlace" color="7" fill="1" visible="no" active="yes"/>
 <layer number="22" name="bPlace" color="7" fill="1" visible="no" active="yes"/>
-<layer number="23" name="tOrigins" color="15" fill="1" visible="no" active="yes"/>
+<layer number="23" name="tOrigins" color="15" fill="1" visible="yes" active="yes"/>
 <layer number="24" name="bOrigins" color="15" fill="1" visible="no" active="yes"/>
 <layer number="25" name="tNames" color="7" fill="1" visible="no" active="yes"/>
@@
 <attribute name="OC_FARNELL" value="1612437" x="13.97" y="15.875" size="1.778" layer="27" rot="R180" display="off"/>
 </element>
-<element name="LED2" library="led" library_urn="urn:adsk.eagle:library:259" package="LED3MM" package3d_urn="urn:adsk.eagle:package:15797/1" value="" x="12.7" y="7.9375" rot="R180">
-<attribute name="MF" value="VISHAY SEMICONDUCTOR" x="12.7" y="7.9375" size="1.778" layer="27" rot="R180" display="off"/>
-<attribute name="OC_FARNELL" value="1612437" x="12.7" y="7.9375" size="1.778" layer="27" rot="R180" display="off"/>
+<element name="LED2" library="led" library_urn="urn:adsk.eagle:library:259" package="LED3MM" package3d_urn="urn:adsk.eagle:package:15797/1" value="" x="13.97" y="7.9375" rot="R180">
+<attribute name="MF" value="VISHAY SEMICONDUCTOR" x="13.97" y="7.9375" size="1.778" layer="27" rot="R180" display="off"/>
+<attribute name="OC_FARNELL" value="1612437" x="13.97" y="7.9375" size="1.778" layer="27" rot="R180" display="off"/>
 </element>
 <element name="R13" library="rcl" library_urn="urn:adsk.eagle:library:334" package="R1206" package3d_urn="urn:adsk.eagle:package:23540/2" value="1k" x="8.89" y="15.875" smashed="yes" rot="MR180">
@@
 <wire x1="21.355" y1="25.4" x2="21.355" y2="25.3175" width="0.4064" layer="1"/>
 <wire x1="21.355" y1="25.4" x2="21.355" y2="21.825" width="0.3048" layer="1"/>
-<wire x1="21.355" y1="21.825" x2="21.59" y2="21.59" width="0.3048" layer="1"/>
-<wire x1="21.59" y1="21.59" x2="21.59" y2="17.932" width="0.3048" layer="1"/>
-<wire x1="21.59" y1="17.932" x2="25.55875" y2="15.23325" width="0.3048" layer="1"/>
 <wire x1="33.655" y1="14.605" x2="25.55875" y2="15.23325" width="0.3048" layer="1"/>
+<wire x1="21.355" y1="21.825" x2="25.55875" y2="17.62125" width="0.3048" layer="1"/>
+<wire x1="25.55875" y1="17.62125" x2="25.55875" y2="15.23325" width="0.3048" layer="1"/>
 </signal>
 <signal name="N$9">
@@
 <contactref element="C1" pad="1"/>
 <contactref element="U2" pad="3"/>
-<wire x1="25.7175" y1="15.9625" x2="27.227" y2="15.9625" width="0.508" layer="16"/>
-<wire x1="27.227" y1="15.9625" x2="28.575" y2="16.0405" width="0.3048" layer="16"/>
-<wire x1="28.575" y1="16.0405" x2="30.0105" y2="16.0405" width="0.508" layer="16"/>
-<wire x1="30.0105" y1="16.0405" x2="30.00375" y2="10.795" width="0.3048" layer="16"/>
-<wire x1="30.00375" y1="10.795" x2="33.655" y2="9.525" width="0.3048" layer="16"/>
+<wire x1="28.575" y1="16.0405" x2="30.3145" y2="16.0405" width="0.4064" layer="16"/>
+<wire x1="30.3145" y1="16.0405" x2="30.32125" y2="16.03375" width="0.4064" layer="16"/>
+<wire x1="30.32125" y1="16.03375" x2="30.32125" y2="11.58875" width="0.4064" layer="16"/>
+<wire x1="32.385" y1="9.525" x2="33.655" y2="9.525" width="0.4064" layer="16"/>
+<wire x1="30.32125" y1="11.58875" x2="32.385" y2="9.525" width="0.4064" layer="16"/>
+<wire x1="28.575" y1="16.0405" x2="25.7955" y2="16.0405" width="0.4064" layer="16"/>
+<wire x1="25.7955" y1="16.0405" x2="25.7175" y2="15.9625" width="0.4064" layer="16"/>
 </signal>
 <signal name="SCK">
@@
 <contactref element="IC1" pad="24"/>
 <contactref element="LED2" pad="A"/>
-<wire x1="13.97" y1="7.9375" x2="18.7325" y2="7.9375" width="0.3048" layer="16"/>
+<wire x1="15.24" y1="7.9375" x2="18.7325" y2="7.9375" width="0.3048" layer="16"/>
 <via x="18.7325" y="7.9375" extent="1-16" drill="0.35" diameter="1.3" shape="octagon"/>
 <wire x1="18.7325" y1="7.9375" x2="20.6375" y2="7.9375" width="0.3048" layer="1"/>
@@
 <contactref element="R14" pad="2"/>
 <wire x1="7.46125" y1="7.94425" x2="7.468" y2="7.9375" width="0.3048" layer="16" curve="90"/>
-<wire x1="7.468" y1="7.9375" x2="11.43" y2="7.9375" width="0.3048" layer="16"/>
+<wire x1="7.468" y1="7.9375" x2="12.7" y2="7.9375" width="0.3048" layer="16"/>
 </signal>
 <signal name="N$17">
