File: PCB/V2A/ESC-simple_V2A.brd (EAGLE design)
At the start: 35.6 x 79.4 mm, 46 parts, among them IC1 MEGA8-AI, IC2 L6369D, IC3 L6369D, IC4 L6369D, IC6 7805T, Q1 SIRC10DP, Q2 SIRC10DP, Q3 SIRC10DP, Q4 SIRC10DP, Q5 SIRC10DP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

Commit message: Added SOFTWARE/Control
Routing:
- net V_BATT: track 69.5 -> 62.3 mm
- net 5V: track 15.0 -> 11.4 mm
Changed lines of the file:
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@@
 <setting verticaltext="up"/>
 </settings>
-<grid distance="0.635" unitdist="mm" unit="mm" style="lines" multiple="1" display="yes" altdistance="6.25" altunitdist="mil" altunit="mil"/>
+<grid distance="50" unitdist="mil" unit="mm" style="lines" multiple="1" display="yes" altdistance="6.25" altunitdist="mil" altunit="mil"/>
 <layers>
 <layer number="1" name="Top" color="4" fill="1" visible="yes" active="yes"/>
@@
 <layer number="14" name="Route14" color="1" fill="6" visible="no" active="no"/>
 <layer number="15" name="Route15" color="4" fill="6" visible="no" active="no"/>
-<layer number="16" name="Bottom" color="1" fill="1" visible="no" active="yes"/>
+<layer number="16" name="Bottom" color="1" fill="1" visible="yes" active="yes"/>
 <layer number="17" name="Pads" color="2" fill="1" visible="yes" active="yes"/>
 <layer number="18" name="Vias" color="2" fill="1" visible="yes" active="yes"/>
-<layer number="19" name="Unrouted" color="6" fill="1" visible="no" active="yes"/>
+<layer number="19" name="Unrouted" color="6" fill="1" visible="yes" active="yes"/>
 <layer number="20" name="Dimension" color="24" fill="1" visible="yes" active="yes"/>
 <layer number="21" name="tPlace" color="7" fill="1" visible="yes" active="yes"/>
-<layer number="22" name="bPlace" color="7" fill="1" visible="no" active="yes"/>
+<layer number="22" name="bPlace" color="7" fill="1" visible="yes" active="yes"/>
 <layer number="23" name="tOrigins" color="15" fill="1" visible="yes" active="yes"/>
-<layer number="24" name="bOrigins" color="15" fill="1" visible="no" active="yes"/>
+<layer number="24" name="bOrigins" color="15" fill="1" visible="yes" active="yes"/>
 <layer number="25" name="tNames" color="7" fill="1" visible="no" active="yes"/>
 <layer number="26" name="bNames" color="7" fill="1" visible="no" active="yes"/>
@@
 <layer number="43" name="vRestrict" color="2" fill="10" visible="no" active="yes"/>
 <layer number="44" name="Drills" color="7" fill="1" visible="no" active="yes"/>
-<layer number="45" name="Holes" color="7" fill="1" visible="no" active="yes"/>
+<layer number="45" name="Holes" color="7" fill="1" visible="yes" active="yes"/>
 <layer number="46" name="Milling" color="3" fill="1" visible="no" active="yes"/>
 <layer number="47" name="Measures" color="7" fill="1" visible="no" active="yes"/>
@@
 <layer number="50" name="dxf" color="7" fill="1" visible="no" active="no"/>
 <layer number="51" name="tDocu" color="7" fill="1" visible="yes" active="yes"/>
-<layer number="52" name="bDocu" color="7" fill="1" visible="no" active="yes"/>
+<layer number="52" name="bDocu" color="7" fill="1" visible="yes" active="yes"/>
 <layer number="53" name="tGND_GNDA" color="7" fill="9" visible="no" active="no"/>
 <layer number="54" name="bGND_GNDA" color="1" fill="9" visible="no" active="no"/>
@@
 </layers>
 <board>
+<fusionsync huburn="a.cGVyc29uYWw6dWUyYWQxMTA4" projecturn="a.cGVyc29uYWw6dWUyYWQxMTA4IzIwMTgwNDA4MTI2NTM4NDc2" f3durn="urn:adsk.wipprod:dm.lineage:grtCamHvQa-VvuCE28b0bg" pcbguid="d24d2f70-779e-44e9-bb75-e6702eb6b2c6" lastpulledtime="" lastsyncedchangeguid="77cf7bea-5ac0-5358-346f-d517b3e4b463"/>
 <plain>
 <wire x1="-17.78" y1="-1.27" x2="17.78" y2="-1.27" width="0" layer="20"/>
@@
 <wire x1="11.43" y1="32.385" x2="13.335" y2="34.29" width="0.508" layer="16"/>
 <wire x1="1.27" y1="32.385" x2="11.43" y2="32.385" width="0.508" layer="16"/>
-<wire x1="13.565" y1="22.455" x2="13.565" y2="24.13" width="0.508" layer="16"/>
-<wire x1="10.16" y1="27.94" x2="13.565" y2="25.17" width="0.508" layer="16"/>
-<wire x1="13.565" y1="25.17" x2="13.565" y2="24.13" width="0.508" layer="16"/>
 <contactref element="C15" pad="+"/>
 <wire x1="11.2" y1="30.48" x2="11.43" y2="30.71" width="0.508" layer="16"/>
@@
 <contactref element="IC6" pad="1"/>
 <wire x1="13.565" y1="24.13" x2="31.115" y2="23.495" width="0" layer="19" extent="16-16"/>
+<wire x1="10.16" y1="27.94" x2="13.565" y2="24.13" width="0" layer="19" extent="1-16"/>
 </signal>
 <signal name="GND">
@@
 <wire x1="14.375" y1="9.525" x2="10.565" y2="13.335" width="0.508" layer="16"/>
 <wire x1="10.565" y1="13.335" x2="10.565" y2="14.605" width="0.508" layer="16"/>
-<wire x1="9.525" y1="17.78" x2="10.565" y2="16.74" width="0.508" layer="16"/>
-<wire x1="10.565" y1="16.74" x2="10.565" y2="14.605" width="0.508" layer="16"/>
 <contactref element="IC6" pad="3"/>
-<wire x1="10.565" y1="16.74" x2="26.035" y2="23.495" width="0" layer="19" extent="16-16"/>
+<wire x1="15.875" y1="9.525" x2="26.035" y2="23.495" width="0" layer="19" extent="1-1"/>
 </signal>
 <signal name="MOSI">
@@
 </note>
 <note version="8.3" severity="warning">
+Since Version 8.3, EAGLE supports Fusion synchronisation.
+This feature will not be available in this version and saving
+the document will break the link to the Fusion PCB feature.
+</note>
+<note version="8.3" severity="warning">

Commit message: V2A Final
V2A already etched.
Parts:
- added R13, R14, R15: 220, rcl:R1206
- added U$1, U$2, U$3: LED, led:3MM_LED
- moved IC6 16.6 mm to (12.1, 11.4), flipped to the bottom
- moved C14 7.62 mm to (12.1, -1.91)
- moved U2 7.62 mm to (12.1, -1.91)
- moved C1 7.31 mm to (0.00, -3.81)
- moved R12 7.31 mm to (0.00, -3.81)
- moved R5 7.30 mm to (3.17, -3.81)
- moved R6 7.30 mm to (3.17, -3.81)
- moved R1 6.85 mm to (-7.62, -2.54), turned to 0 degrees
- moved C12 3.42 mm to (13.3, 17.8), flipped to the top
- moved J1 1.91 mm to (-12.1, 6.99)
- moved C13 1.80 mm to (10.8, 25.4), turned to 180 degrees
- moved C2 1.62 mm to (-7.62, 4.45), turned to 0 degrees
- moved Y1 1.27 mm to (-6.38, 14.4)
- moved C4 1.27 mm to (-1.27, 18.4)
- moved C5 1.27 mm to (-11.4, 18.4)
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Connections:
- removed net PB1: IC1.13
- removed net PB2: IC1.14
- removed net PC0: IC1.23
- removed net PC1: IC1.24
- removed net PC2: IC1.25
- removed net SCL: IC1.28
- removed net SDA: IC1.27
- new net N$14: R14.1, U$2.A
- new net N$15: R13.1, U$1.A
- new net N$17: R15.1, U$3.A
- new net TEST_PIN_1: IC1.23, R13.2
- new net TEST_PIN_2: IC1.24, R14.2
- net 5V: now also R15.2
- net CONTROL: now also IC1.12; no longer IC1.32
- net GND: now also U$1.C, U$2.C, U$3.C
- net ZC_B: now also IC1.13; no longer IC1.12
Routing:
- net ZC_C: track 40.1 -> 29.4 mm
- net V_BATT: track 62.3 -> 73.0 mm, vias 9 -> 12
- net SCL: track 10.5 -> 0.00 mm, vias 1 -> 0
- net GND: track 57.8 -> 68.1 mm, vias 5 -> 3
- net SDA: track 9.25 -> 0.00 mm, vias 1 -> 0
- net CURRENT: track 19.4 -> 28.5 mm
- net PB1: track 8.91 -> 0.00 mm, vias 1 -> 0
- net PB2: track 8.33 -> 0.00 mm, vias 1 -> 0
- net N$15: track 0.00 -> 6.55 mm
- net RST: track 10.8 -> 17.3 mm
- net N$14: track 0.00 -> 6.37 mm
- net TEST_PIN_2: track 0.00 -> 6.31 mm
- net N$17: track 0.00 -> 5.72 mm
- net ZC_B: track 46.6 -> 51.9 mm
- net 5V: track 11.4 -> 15.3 mm, vias 0 -> 1
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Other:
- board size 35.6 x 79.4 mm -> 35.6 x 87 mm
- board text added: "ESC V2A"
