File: PCB/V2A/ESC-simple_V2A.sch (EAGLE design)
At the start: 46 parts, among them IC1 MEGA8-AI, IC2 L6369D, IC3 L6369D, IC4 L6369D, IC6 7805T, Q1 SIRC10DP, Q2 SIRC10DP, Q3 SIRC10DP, Q4 SIRC10DP, Q5 SIRC10DP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

Commit message: V2A Final
V2A already etched.
Parts:
- added R13, R14, R15: 220, rcl:R-EU_R1206
- added U$1, U$2, U$3: LED, led:LED
Connections:
- removed net PB1: IC1.PB1(OC1A)
- removed net PB2: IC1.PB2(SS/OC1B)
- removed net PC0: IC1.PC0(ADC0)
- removed net PC1: IC1.PC1(ADC1)
- removed net PC2: IC1.PC2(ADC2)
- removed net SCL: IC1.PC5(ADC5/SCL)
- removed net SDA: IC1.PC4(ADC4/SDA)
- new net N$14: R14.1, U$2.A
- new net N$15: R13.1, U$1.A
- new net N$17: R15.1, U$3.A
- new net TEST_PIN_1: IC1.PC0(ADC0), R13.2
- new net TEST_PIN_2: IC1.PC1(ADC1), R14.2
- net 5V: now also R15.2
- net CONTROL: now also IC1.PB0(ICP); no longer IC1.PD2(INT0)
- net GND: now also U$1.C, U$2.C, U$3.C
- net ZC_B: now also IC1.PB1(OC1A); no longer IC1.PB0(ICP)
Other:
- moved on the sheet: C12, C13, C14, C15, IC6, PAD4, PAD5, U2G2, U2G3
